File: Charger&Bost_MP2637/$MP2637.sch (KiCad schematic (older format))
At the start: 45 parts

Commit message: MP2637: засстановка компонентов...
Parts:
- GB1: footprint Connectors:for_PolarOut_PLL1.27-2 -> Connectors:for_PolarOut_PLS-2
- XP3: footprint Connectors:PLS2-2 -> Connectors:PLS-2
Changed lines of the file:
@@
 F 0 "XP3" H 650 5900 60  0000 C CNN
 F 1 "NTC" V 1000 5550 60  0000 C CNN
-F 2 "Connectors:PLS2-2" H 650 5300 60  0001 C CNN
+F 2 "Connectors:PLS-2" H 650 5300 60  0001 C CNN
 F 3 "" H 900 5750 60  0000 C CNN
 F 4 "0" H 450 5900 60  0001 C CNN "SolderPoints"
@@
 F 0 "GB1" H 9550 1550 60  0000 L CNN
 F 1 "Li-ion" H 9550 1450 60  0000 L CNN
-F 2 "Connectors:for_PolarOut_PLL1.27-2" H 9550 1350 60  0001 L CNN
+F 2 "Connectors:for_PolarOut_PLS-2" H 9550 1350 60  0001 L CNN
 F 3 "" H 9350 1700 60  0000 C CNN
 F 4 "0" H 9250 1650 60  0001 C CNN "SolderPoints"
