File: MagneticSwitch_AS-V20&AS-M15/AS-V20_AS-M15_simple.kicad_pcb (KiCad board)
At the start: 2 copper layers, 9 x 6 mm, 5 parts

Commit message: + AS-V20_AS-M15_invert_cover
Parts:
- Logo1: moved to F.Cu
