File: Backlight_WS2813/WS2813_single.sch (KiCad schematic (older format))
At the start: 5 parts

Commit message: вариант WS2813_single: с обжимными разъёмамы "плата-провод" (начата работа)
Parts:
- HL1: symbol WS2813 -> LED:WS2813
- Hole1: symbol HoleMetalled -> PCB_details:HoleMetalled
- Logo1: symbol Eldalim -> Graphics:Eldalim
- XP1, XP2: footprint Connectors:FlatConn-4_1,27 -> Connectors:for_WS2813_AVX_00-9176; symbol for_WS2813 -> Connectors:for_WS2813
Other:
- moved on the sheet: HL1, Hole1, XP1, XP2
