File: Backlight_WS2813/WS2813_single_for_wire.kicad_pcb (KiCad board)
At the start: 2 copper layers, 10 x 14.8 mm, 4 parts

Commit message: .
Parts:
- moved XP1 1.00 mm to (96.0, 50.0)
- moved XP2 1.00 mm to (104.0, 50.0)
Other:
- board size 10 x 14.8 mm -> 12 x 17.7 mm
Changed lines of the file:
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@@
   (general
     (thickness 1.6)
-    (drawings 25)
+    (drawings 29)
     (tracks 0)
     (zones 0)
@@
       (effects (font (size 0.6 0.6) (thickness 0.15)))
     )
-    (fp_text user . (at 3.1 3 270) (layer F.SilkS)
+    (fp_line (start -2.5 -2.5) (end 2.5 -2.5) (layer F.SilkS) (width 0.14986))
+    (fp_line (start -2.5 2.5) (end -2.5 -2.5) (layer F.SilkS) (width 0.15))
+    (fp_line (start 2.5 2.5) (end -2.5 2.5) (layer F.SilkS) (width 0.15))
+    (fp_line (start 2.5 -2.5) (end 2.5 2.5) (layer F.SilkS) (width 0.15))
+    (fp_circle (center 0 0) (end 0 2.2) (layer F.SilkS) (width 0.15))
+    (fp_line (start 2.5 1.6) (end 1.6 2.5) (layer F.SilkS) (width 0.15))
+    (fp_line (start 1.7 2.5) (end 2.5 1.7) (layer F.SilkS) (width 0.15))
+    (fp_line (start 2.5 1.9) (end 1.9 2.5) (layer F.SilkS) (width 0.15))
+    (fp_line (start 2.1 2.5) (end 2.5 2.1) (layer F.SilkS) (width 0.15))
+    (fp_line (start 2.5 2.3) (end 2.3 2.5) (layer F.SilkS) (width 0.15))
+    (fp_line (start 1.5 2.5) (end 2.5 1.5) (layer F.SilkS) (width 0.15))
+    (fp_text user . (at 2.4 2.8 270 unlocked) (layer F.SilkS)
       (effects (font (size 2 2) (thickness 0.5)))
     )
-    (fp_line (start 1.5 2.5) (end 2.5 1.5) (layer F.SilkS) (width 0.15))
-    (fp_line (start 2.5 2.3) (end 2.3 2.5) (layer F.SilkS) (width 0.15))
-    (fp_line (start 2.1 2.5) (end 2.5 2.1) (layer F.SilkS) (width 0.15))
-    (fp_line (start 2.5 1.9) (end 1.9 2.5) (layer F.SilkS) (width 0.15))
-    (fp_line (start 1.7 2.5) (end 2.5 1.7) (layer F.SilkS) (width 0.15))
-    (fp_line (start 2.5 1.6) (end 1.6 2.5) (layer F.SilkS) (width 0.15))
-    (fp_circle (center 0 0) (end 0 2.2) (layer F.SilkS) (width 0.15))
-    (fp_line (start 2.5 -2.5) (end 2.5 2.5) (layer F.SilkS) (width 0.15))
-    (fp_line (start 2.5 2.5) (end -2.5 2.5) (layer F.SilkS) (width 0.15))
-    (fp_line (start -2.5 2.5) (end -2.5 -2.5) (layer F.SilkS) (width 0.15))
-    (fp_line (start -2.5 -2.5) (end 2.5 -2.5) (layer F.SilkS) (width 0.14986))
-    (pad 5 smd oval (at -2.5 0 180) (size 1.6 1.1) (layers F.Cu F.Mask)
+    (pad 3 smd oval (at 2.5 -1.6 180) (size 1.6 1.1) (layers F.Cu F.Paste F.Mask)
+      (net 5 /Dout))
+    (pad 6 smd oval (at -2.5 1.6 180) (size 1.6 1.1) (layers F.Cu F.Paste F.Mask)
+      (net 4 /BDin))
+    (pad 4 smd oval (at -2.5 -1.6 180) (size 1.6 1.1) (layers F.Cu F.Paste F.Mask)
+      (net 3 /Din))
+    (pad 1 smd rect (at 2.5 1.6 180) (size 1.6 1.1) (layers F.Cu F.Paste F.Mask)
+      (net 2 +VCC))
+    (pad 2 smd oval (at 2.5 0 180) (size 1.6 1.1) (layers F.Cu F.Paste F.Mask)
+      (net 2 +VCC))
+    (pad 5 smd oval (at -2.5 0 180) (size 1.6 1.1) (layers F.Cu F.Paste F.Mask)
       (net 1 GND))
-    (pad 2 smd oval (at 2.5 0 180) (size 1.6 1.1) (layers F.Cu F.Mask)
-      (net 2 +VCC))
-    (pad 1 smd rect (at 2.5 1.6 180) (size 1.6 1.1) (layers F.Cu F.Mask)
-      (net 2 +VCC))
-    (pad 4 smd oval (at -2.5 -1.6 180) (size 1.6 1.1) (layers F.Cu F.Mask)
-      (net 3 /Din))
-    (pad 6 smd oval (at -2.5 1.6 180) (size 1.6 1.1) (layers F.Cu F.Mask)
-      (net 4 /BDin))
-    (pad 3 smd oval (at 2.5 -1.6 180) (size 1.6 1.1) (layers F.Cu F.Mask)
-      (net 5 /Dout))
   )
   (module PCB_details:Hole_for_M2 (layer F.Cu)
@@
   )
   (module Connectors:for_WS2813_AVX_00-9176 (layer B.Cu)
-    (at 97 50 270)
-    (fp_text reference XP1 (at -0.25 3.25 270) (layer B.SilkS)
+    (at 96 50 270)
+    (fp_text reference XP1 (at -0.25 3.25 270) (layer B.SilkS) hide
       (effects (font (size 0.6 0.6) (thickness 0.15)) (justify mirror))
     )
-    (fp_text value IN (at -0.25 2.5 90) (layer B.SilkS)
-      (effects (font (size 0.6 0.6) (thickness 0.15)) (justify mirror))
+    (fp_text value IN (at 7.5 -1.25 180) (layer B.SilkS)
+      (effects (font (size 0.8 0.8) (thickness 0.15)) (justify mirror))
     )
     (fp_text user BDAT (at 4.75 2.75 90) (layer B.SilkS) hide
       (effects (font (size 1 0.8) (thickness 0.15)) (justify mirror))
     )
-    (fp_text user 1 (at -7.5 0 270) (layer B.SilkS)
+    (fp_text user 1 (at -7.25 -1 270) (layer B.SilkS)
       (effects (font (size 1.8 1) (thickness 0.15)) (justify mirror))
     )
@@
   )
   (module Connectors:for_WS2813_AVX_00-9176 (layer B.Cu)
-    (at 103 50 270)
-    (fp_text reference XP2 (at 0 -2.5 270) (layer B.SilkS)
+    (at 104 50 270)
+    (fp_text reference XP2 (at 0 -2.5 270) (layer B.SilkS) hide
       (effects (font (size 0.6 0.6) (thickness 0.15)) (justify mirror))
     )
-    (fp_text value OUT (at 0 -3.5 90) (layer B.SilkS)
-      (effects (font (size 0.6 0.6) (thickness 0.15)) (justify mirror))
-    )
-    (fp_text user DAT (at 2 3 90) (layer B.SilkS)
-      (effects (font (size 1 0.8) (thickness 0.15)) (justify mirror))
-    )
-    (fp_text user GND (at -2.5 3 90) (layer B.SilkS)
-      (effects (font (size 1 0.8) (thickness 0.15)) (justify mirror))
-    )
-    (fp_text user VCC (at -5.25 3 90) (layer B.SilkS)
-      (effects (font (size 1 0.8) (thickness 0.15)) (justify mirror))
+    (fp_text value OUT (at 7.5 0.75 180) (layer B.SilkS)
+      (effects (font (size 0.8 0.8) (thickness 0.15)) (justify mirror))
+    )
+    (fp_text user DAT (at 2 4 180) (layer B.SilkS)
+      (effects (font (size 1.5 1.2) (thickness 0.2)) (justify mirror))
+    )
+    (fp_text user GND (at -2 4 180) (layer B.SilkS)
+      (effects (font (size 1.5 1.2) (thickness 0.2)) (justify mirror))
+    )
+    (fp_text user VCC (at -5 4 180) (layer B.SilkS)
+      (effects (font (size 1.5 1.2) (thickness 0.2)) (justify mirror))
     )
     (fp_line (start 6.65 -1.85) (end -6.05 -1.85) (layer B.SilkS) (width 0.15))
@@
     (fp_line (start -6.05 -1.85) (end -6.65 -1.25) (layer B.SilkS) (width 0.15))
     (fp_line (start -6.65 -1.25) (end -6.65 1.25) (layer B.SilkS) (width 0.15))
-    (fp_text user 1 (at -7.5 0 270) (layer B.SilkS)
+    (fp_text user 1 (at -7.25 1 270) (layer B.SilkS)
       (effects (font (size 1.8 1) (thickness 0.15)) (justify mirror))
     )
-    (fp_text user BDAT (at 4.5 3 270) (layer B.SilkS)
-      (effects (font (size 1 0.8) (thickness 0.15)) (justify mirror))
+    (fp_text user BDAT (at 5 4) (layer B.SilkS)
+      (effects (font (size 1.5 1.2) (thickness 0.2)) (justify mirror))
     )
     (pad 1 smd rect (at -4.8 0 270) (size 2.5 2.7) (layers B.Cu B.Paste B.Mask)
@@
       (net 3 /Din))
   )
-  (gr_arc (start 100 49) (end 95 44) (angle 90) (layer Edge.Cuts) (width 0.15))
-  (gr_line (start 95 56.75) (end 95 44) (angle 90) (layer Edge.Cuts) (width 0.15))
-  (gr_line (start 105 56.75) (end 105 44) (angle 90) (layer Edge.Cuts) (width 0.15))
-  (gr_line (start 95 56.75) (end 105 56.75) (angle 90) (layer Edge.Cuts) (width 0.15))
-  (gr_line (start 100.4 56.65) (end 100.8 56.25) (angle 90) (layer B.SilkS) (width 0.2))
-  (gr_line (start 100.4 55.85) (end 100.4 56.65) (angle 90) (layer B.SilkS) (width 0.2))
-  (gr_line (start 100.5 56.55) (end 100.5 55.95) (angle 90) (layer B.SilkS) (width 0.15))
-  (gr_line (start 100.8 56.25) (end 100.4 55.85) (angle 90) (layer B.SilkS) (width 0.2))
-  (gr_line (start 100.7 56.25) (end 99.2 56.25) (angle 90) (layer B.SilkS) (width 0.25))
-  (gr_line (start 99.35 42.65) (end 100.65 42.65) (angle 90) (layer B.SilkS) (width 0.25))
-  (gr_line (start 100.45 42.35) (end 100.45 42.95) (angle 90) (layer B.SilkS) (width 0.15))
+  (gr_line (start 98.75 57) (end 101 57) (angle 90) (layer B.SilkS) (width 0.3))
+  (gr_line (start 101.25 57) (end 100.5 57.5) (angle 90) (layer B.SilkS) (width 0.15))
+  (gr_line (start 100.5 57.5) (end 100.75 57) (angle 90) (layer B.SilkS) (width 0.15))
+  (gr_line (start 101.25 57) (end 100.5 56.5) (angle 90) (layer B.SilkS) (width 0.15))
+  (gr_line (start 100.5 56.5) (end 100.75 57) (angle 90) (layer B.SilkS) (width 0.15))
+  (gr_line (start 100.75 57.25) (end 101 57) (angle 90) (layer B.SilkS) (width 0.15))
+  (gr_line (start 101 57) (end 100.75 56.75) (angle 90) (layer B.SilkS) (width 0.15))
+  (gr_line (start 101 43) (end 100.75 42.75) (angle 90) (layer B.SilkS) (width 0.15))
+  (gr_line (start 100.75 43.25) (end 101 43) (angle 90) (layer B.SilkS) (width 0.15))
+  (gr_line (start 100.5 42.5) (end 100.75 43) (angle 90) (layer B.SilkS) (width 0.15))
+  (gr_line (start 101.25 43) (end 100.5 42.5) (angle 90) (layer B.SilkS) (width 0.15))
+  (gr_line (start 100.5 43.5) (end 100.75 43) (angle 90) (layer B.SilkS) (width 0.15))
+  (gr_line (start 101.25 43) (end 100.5 43.5) (angle 90) (layer B.SilkS) (width 0.15))
+  (gr_line (start 98.75 43) (end 101 43) (angle 90) (layer B.SilkS) (width 0.3))
+  (gr_arc (start 100 50.75) (end 106 56.75) (angle 90) (layer Edge.Cuts) (width 0.15))
+  (gr_arc (start 100 50) (end 94 44) (angle 90) (layer Edge.Cuts) (width 0.15))
+  (gr_line (start 94 56.75) (end 94 44) (angle 90) (layer Edge.Cuts) (width 0.15))
+  (gr_line (start 106 56.75) (end 106 44) (angle 90) (layer Edge.Cuts) (width 0.15))
   (gr_text eldalim (at 100 56.05) (layer F.SilkS)
     (effects (font (size 0.7 0.7) (thickness 0.15) italic))
   )
-  (gr_line (start 100.35 43.05) (end 100.75 42.65) (angle 90) (layer B.SilkS) (width 0.2))
-  (gr_line (start 100.35 42.25) (end 100.35 43.05) (angle 90) (layer B.SilkS) (width 0.2))
-  (gr_line (start 100.75 42.65) (end 100.35 42.25) (angle 90) (layer B.SilkS) (width 0.2))
   (gr_line (start 141 57.5) (end 143 57.5) (angle 90) (layer Dwgs.User) (width 0.15))
   (gr_line (start 141.25 57.25) (end 141 57.5) (angle 90) (layer Dwgs.User) (width 0.15))
