File: Charger_MP2611/MP2611.sch (KiCad schematic (older format))
At the start: 33 parts

Commit message: обновлён MP2611
Parts:
- C1, C4, C7: symbol C_0603 -> Capacitors:C_0603
- C2, C3, C5, C6: symbol C_0805 -> Capacitors:C_0805
- DA1: symbol MP2611 -> Chargers:MP2611
- GB1: symbol BATT -> MP2611-rescue:BATT
- HL1, HL2, HL3: symbol LED_0603 -> LED:LED_0603
- HOLE1, HOLE2: symbol HOLE_METALLED -> MP2611-rescue:HOLE_METALLED
- L1: symbol Inductor -> Inductors:Inductor
- Label1: symbol Eldalim -> Graphics:Eldalim
- R1, R2, R3, R4, R5, R9: symbol R_0603 -> Resistors:R_0603
- R6: symbol R_0805 -> Resistors:R_0805
- R7, R8: symbol R_1206 -> Resistors:R_1206
- VT1: symbol IRLML2502 -> Transistors:IRLML2502
- XP1, XP2, XP4: symbol conn-1p -> MP2611-rescue:conn-1p
- XP3: symbol conn-2p -> MP2611-rescue:conn-2p
- XS1, XS2: symbol mcro/mini-USB -> MP2611-rescue:mcro_mini-USB
- fuse1: symbol FuseX2 -> MP2611-rescue:FuseX2
