File: Charger_MP2611/MP2611.kicad_pcb (KiCad board)
At the start: 2 copper layers, 42.9 x 17.3 mm, 33 parts

Commit message: обновлён MP2611
Parts:
- XS2: footprint Connectors:USB-micro_B -> Connectors:USB-micro_B+Hole
- moved XS2 0.07 mm to (89.1, 59.9)

Commit message: MP2611 - обновлён контур платы
Parts:
- Label1: footprint Graphics:Eldalim_17x15_back -> Graphics:Eldalim_17x15
- moved Label1 2.72 mm to (112.6, 59.8), turned to 0 degrees
Other:
- board size 42.9 x 17.3 mm -> 43 x 17.3 mm

Commit message: MP2611: переход на KiCad 7 + комментарий в схеме
Other:
- net class Default removed
- net class wide removed
- net class wide wide removed
