File: Buck_MP8765/MP8765.kicad_pcb (KiCad board)
At the start: 2 copper layers, 40 x 20 mm, 28 parts, among them J1 Jumper

Commit message: + результаты тестов и правки
Parts:
- R7: value 130k -> 150k
Other:
- board text added: "EN PG"
- board text removed: "PG EN"
Changed lines of the file:
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@@
       (effects (font (size 0.6 0.6) (thickness 0.15)))
     )
-    (fp_text value 130k (at -1.225 1.475) (layer F.SilkS)
+    (fp_text value 150k (at -1.225 1.475) (layer F.SilkS)
       (effects (font (size 0.6 0.6) (thickness 0.15)))
     )
@@
     )
   )
-  (gr_text "PG  EN" (at 127 53.4) (layer F.SilkS)
+  (gr_text "EN  PG" (at 127 53.5) (layer F.SilkS)
     (effects (font (size 0.8 0.8) (thickness 0.15)))
   )
