File: TouchSensor_AT42QT1011/AT42QT1011.sch (KiCad schematic (older format))
At the start: 13 parts

Commit message: Переоткрыты схемы
Parts:
- C1: symbol C_0805 -> Capacitors:C_0805
- C2: symbol C_0603 -> Capacitors:C_0603
- DA1: symbol AT42QT1011 -> Sensors:AT42QT1011
- E1: symbol SENS -> AT42QT1011-rescue:SENS
- HL1: symbol LED_0603 -> LED:LED_0603
- HOLE1, HOLE2: symbol HOLE_METALLED -> AT42QT1011-rescue:HOLE_METALLED
- Logo1: symbol Eldalim -> Graphics:Eldalim
- R1: symbol R_0805 -> Resistors:R_0805
- R2: symbol R_0603 -> Resistors:R_0603
- XP1: symbol for_SENS -> AT42QT1011-rescue:for_SENS
- XP2: symbol conn-1p -> AT42QT1011-rescue:conn-1p
- fuse1: symbol FuseX2 -> AT42QT1011-rescue:FuseX2
Changed lines of the file:
@@
-EESchema Schematic File Version 2
-LIBS:Audio
-LIBS:Capacitors
-LIBS:Chargers
-LIBS:Connektors
-LIBS:CPU
-LIBS:DC-DC
-LIBS:Drivers
-LIBS:Inductors
-LIBS:LED
-LIBS:Opto
-LIBS:OU
-LIBS:PCB details
-LIBS:Quartz
-LIBS:Regulators
-LIBS:Resistors
-LIBS:Sensors
-LIBS:Sound
-LIBS:Switches
-LIBS:Logic
-LIBS:Diodes
-LIBS:Transistors
-LIBS:Interface
-LIBS:Modules
-LIBS:Radio
-LIBS:Relays
-LIBS:Graphics
-LIBS:Motors
-LIBS:Power
-LIBS:power
-LIBS:AT42QT1011-cache
-EELAYER 24 0
+EESchema Schematic File Version 4
+EELAYER 30 0
 EELAYER END
 $Descr A4 11693 8268
@@
 NoConn ~ 18450 -1450
 $Comp
-L Eldalim Logo1
+L Graphics:Eldalim Logo1
 U 1 1 57C01481
 P 1750 3200
@@
 $EndComp
 $Comp
-L HOLE_METALLED HOLE2
+L AT42QT1011-rescue:HOLE_METALLED HOLE2
 U 1 1 57CD4EB6
 P 5800 3400
@@
 	6150 3400 6200 3400
 $Comp
-L HOLE_METALLED HOLE1
+L AT42QT1011-rescue:HOLE_METALLED HOLE1
 U 1 1 57CD4EC5
 P 5800 3050
@@
 	6150 3050 6200 3050
 $Comp
-L AT42QT1011 DA1
+L Sensors:AT42QT1011 DA1
 U 1 1 57D18E63
 P 3550 1750
@@
 $EndComp
 $Comp
-L SENS E1
+L AT42QT1011-rescue:SENS E1
 U 1 1 57D18E71
 P 1400 1450
@@
 $EndComp
 $Comp
-L GND #U01
+L Power:GND #U01
 U 1 1 57D18E78
 P 4200 2500
@@
 $EndComp
 $Comp
-L GND #U02
+L Power:GND #U02
 U 1 1 57D18E7E
 P 4700 2500
@@
 $EndComp
 $Comp
-L C_0805 C1
+L Capacitors:C_0805 C1
 U 1 1 57D18E8A
 P 2850 1800
@@
 $EndComp
 $Comp
-L GND #U03
+L Power:GND #U03
 U 1 1 57D18EA0
 P 5300 2500
@@
 VCC
 $Comp
-L PWR_FLAG #FLG04
+L Power:PWR_FLAG #FLG04
 U 1 1 57D18EB1
 P 4700 1300
@@
 $EndComp
 $Comp
-L PWR_FLAG #FLG05
+L Power:PWR_FLAG #FLG05
 U 1 1 57D18EDD
 P 4500 3400
@@
 $EndComp
 $Comp
-L GND #U06
+L Power:GND #U06
 U 1 1 57D18EE3
 P 4500 3400
@@
 	3000 2050 2850 2050
 Wire Wire Line
-	2700 1450 3000 1450
+	2700 1450 2850 1450
 Wire Wire Line
 	2850 1550 2850 1450
@@
 	1900 1450 1750 1450
 Wire Wire Line
-	4700 1300 4700 1750
-Wire Wire Line
-	4100 1450 5550 1450
+	4700 1300 4700 1450
+Wire Wire Line
+	4100 1450 4700 1450
 Wire Wire Line
 	4700 2250 4700 2500
@@
 	4200 2050 4100 2050
 $Comp
-L R_0805 R1
+L Resistors:R_0805 R1
 U 1 1 57D19022
 P 2300 1450
@@
 $EndComp
 $Comp
-L for_SENS XP1
+L AT42QT1011-rescue:for_SENS XP1
 U 1 1 57D19428
 P 5850 1650
@@
 $EndComp
 $Comp
-L FuseX2 fuse1
+L AT42QT1011-rescue:FuseX2 fuse1
 U 1 1 57D1956E
 P 3250 3250
@@
 	3650 3250 3650 3400
 $Comp
-L GND #U07
+L Power:GND #U07
 U 1 1 57D1996C
 P 3650 3400
@@
 mode
 $Comp
-L conn-1p XP2
+L AT42QT1011-rescue:conn-1p XP2
 U 1 1 57D1A1C8
 P 6000 2300
@@
 NoConn ~ 6200 3400
 $Comp
-L LED_0603 HL1
+L LED:LED_0603 HL1
 U 1 2 57D403F9
 P 3200 2600
@@
 $EndComp
 $Comp
-L R_0603 R2
+L Resistors:R_0603 R2
 U 1 1 57D40400
 P 2400 2600
@@
 	3700 2600 3600 2600
 $Comp
-L GND #U08
+L Power:GND #U08
 U 1 1 57D404FB
 P 3700 2600
@@
 Out
 $Comp
-L C_0603 C2
+L Capacitors:C_0603 C2
 U 1 1 57D445EF
 P 4700 2000
@@
 	1    0    0    -1
 $EndComp
+Wire Wire Line
+	2850 1450 3000 1450
+Wire Wire Line
+	4700 1450 4700 1750
+Wire Wire Line
+	4700 1450 5550 1450
 $EndSCHEMATC
