File: LowPower Light-sensor/LP_Light-sensor.kicad_pcb (KiCad board)
At the start: 2 copper layers, 25 x 15 mm, 26 parts

Commit message: Датчик освещённости: работа завершена
Parts:
- C3, C6: value 0.1uF -> 0.1u
- C7: value 10uF -> 10u
- R1, R4: value 100k -> 10M
- R3: value 100k -> 1M
- R5: value 1M -> 10M
- moved Hole1 0.50 mm to (105.0, 62.2)
- moved Hole2 0.50 mm to (105.0, 52.8)
- moved C1 0.25 mm to (112.8, 55.0)
- moved DA1 0.25 mm to (112.8, 57.2)
- moved R2 0.25 mm to (112.8, 53.2)
Routing:
- net GND: track 0.00 -> 108.5 mm, vias 0 -> 18
- net /+LightSns_PWR: track 0.00 -> 35.0 mm
- net /LightSns_OUT: track 0.00 -> 21.7 mm, vias 0 -> 2
- net GNDP: track 0.00 -> 19.2 mm, vias 0 -> 1
- net /LightSns_Sign: track 0.00 -> 14.7 mm, vias 0 -> 1
- net +VCC: track 0.00 -> 13.4 mm
- net Net-(R1-Pad2): track 0.00 -> 12.9 mm, vias 0 -> 2
- net Net-(C1-Pad1): track 0.00 -> 9.67 mm
- net Net-(HL1-PadA): track 0.00 -> 4.42 mm, vias 0 -> 1
- added copper zone on B.Cu, net GND
- added copper zone on F.Cu, net GND
Other:
- board text added: "Light-sensor"
- board text removed: "Low-Power Light-sensor"
