File: LowPower Light-sensor/LP_Light-sensor.sch (KiCad schematic (older format))
At the start: 26 parts

Commit message: Датчик освещённости: работа завершена
Parts:
- C3, C6: value 0.1uF -> 0.1u
- C7: value 10uF -> 10u
- R1, R4: value 100k -> 10M
- R3: value 100k -> 1M
- R5: value 1M -> 10M
Other:
- note added: "Light-sensor"
- note removed: "Low-Power Light-sensor"
- moved on the sheet: C1, C3, C4, C5, DA1, R2
Changed lines of the file:
@@
 Connection ~ 5400 7400
 Text Notes 7050 6875 0    197  ~ 0
-Low-Power Light-sensor
+Light-sensor
 $Comp
 L Protection:BLM18AG102 L1
@@
 P 8300 4700
 F 0 "C7" H 8450 4900 60  0000 C CNN
-F 1 "10uF" H 8450 4800 60  0000 C CNN
+F 1 "10u" H 8450 4800 60  0000 C CNN
 F 2 "Capacitors:CAP0603" H 8500 4600 60  0001 C CNN
 F 3 "" H 8300 4950 60  0000 C CNN
@@
 P 6700 4700
 F 0 "C6" H 6850 4900 60  0000 C CNN
-F 1 "0.1uF" H 6850 4800 60  0000 C CNN
+F 1 "0.1u" H 6850 4800 60  0000 C CNN
 F 2 "Capacitors:CAP0603" H 6900 4600 60  0001 C CNN
 F 3 "" H 6700 4950 60  0000 C CNN
@@
 U 1 2 6335948D
 P 4950 1750
-F 0 "R4" H 4950 2000 60  0000 C CNN
-F 1 "100k" H 4950 1900 60  0000 C CNN
+F 0 "R4" H 4900 2000 60  0000 C CNN
+F 1 "10M" H 4900 1900 60  0000 C CNN
 F 2 "Resistors:RES0603" H 4950 1600 60  0001 C CNN
 F 3 "" H 4550 1750 60  0000 C CNN
@@
 	3850 2450 3850 2400
 Wire Wire Line
-	5200 2000 5150 2000
+	5250 2000 5200 2000
 Connection ~ 4700 2000
 Wire Wire Line
@@
 Connection ~ 4200 2400
 Wire Wire Line
-	4200 2400 5200 2400
+	4200 2400 5250 2400
 Wire Wire Line
 	4200 2400 4200 2600
 Wire Wire Line
-	5450 1050 5150 1050
+	5500 1050 5200 1050
 $Comp
 L Capacitors:C_0603 C1
 U 1 2 633594BB
-P 5750 1050
-F 0 "C1" H 5900 1250 60  0000 C CNN
-F 1 "10nF" H 5900 1150 60  0000 C CNN
-F 2 "Capacitors:CAP0603" H 5950 950 60  0001 C CNN
-F 3 "" H 5750 1300 60  0000 C CNN
-F 4 "2" H 5650 1250 60  0001 C CNN "SolderPoints"
-F 5 "0" H 5650 1150 60  0001 C CNN "SolderPoints_DIP"
-F 6 "0603" H 5800 950 60  0001 L CNN "Size"
-	1    5750 1050
+P 5800 1050
+F 0 "C1" H 5950 1250 60  0000 C CNN
+F 1 "10nF" H 5950 1150 60  0000 C CNN
+F 2 "Capacitors:CAP0603" H 6000 950 60  0001 C CNN
+F 3 "" H 5800 1300 60  0000 C CNN
+F 4 "2" H 5700 1250 60  0001 C CNN "SolderPoints"
+F 5 "0" H 5700 1150 60  0001 C CNN "SolderPoints_DIP"
+F 6 "0603" H 5850 950 60  0001 L CNN "Size"
+	1    5800 1050
 	1    0    0    -1
 $EndComp
@@
 U 1 2 633594D3
 P 4100 1750
-F 0 "R3" H 4100 2000 60  0000 C CNN
-F 1 "100k" H 4100 1900 60  0000 C CNN
+F 0 "R3" H 4050 2000 60  0000 C CNN
+F 1 "1M" H 4050 1900 60  0000 C CNN
 F 2 "Resistors:RES0603" H 4100 1600 60  0001 C CNN
 F 3 "" H 3700 1750 60  0000 C CNN
@@
 P 4950 3000
 F 0 "R5" H 4900 3250 60  0000 C CNN
-F 1 "1M" H 4900 3150 60  0000 C CNN
+F 1 "10M" H 4900 3150 60  0000 C CNN
 F 2 "Resistors:RES0603" H 4950 2850 60  0001 C CNN
 F 3 "" H 4550 3000 60  0000 C CNN
@@
 $EndComp
 Wire Wire Line
-	5300 1550 5150 1550
-Wire Wire Line
-	6250 1550 6100 1550
+	5350 1550 5200 1550
+Wire Wire Line
+	6300 1550 6150 1550
 $Comp
 L Resistors:R_0603 R2
 U 1 1 63359500
-P 5700 1550
-F 0 "R2" H 5700 1800 60  0000 C CNN
-F 1 "47k" H 5700 1700 60  0000 C CNN
-F 2 "Resistors:RES0603" H 5700 1400 60  0001 C CNN
-F 3 "" H 5300 1550 60  0000 C CNN
-F 4 "2" H 5500 1800 60  0001 C CNN "SolderPoints"
-F 5 "0" H 5500 1700 60  0001 C CNN "SolderPoints_DIP"
-F 6 "0603" H 5700 1550 60  0001 C CNN "Case"
-	1    5700 1550
+P 5750 1550
+F 0 "R2" H 5750 1800 60  0000 C CNN
+F 1 "47k" H 5750 1700 60  0000 C CNN
+F 2 "Resistors:RES0603" H 5750 1400 60  0001 C CNN
+F 3 "" H 5350 1550 60  0000 C CNN
+F 4 "2" H 5550 1800 60  0001 C CNN "SolderPoints"
+F 5 "0" H 5550 1700 60  0001 C CNN "SolderPoints_DIP"
+F 6 "0603" H 5750 1550 60  0001 C CNN "Case"
+	1    5750 1550
 	1    0    0    -1
 $EndComp
@@
 L OU:TLV3691 DA1
 U 1 1 633C251E
-P 5700 2200
-F 0 "DA1" H 5700 2650 60  0000 C CNN
-F 1 "TLV3691" H 5700 2550 60  0000 C CNN
-F 2 "SOT,_TO:SOT353" H 5700 1850 60  0001 C CNN
-F 3 "" H 5700 1850 60  0000 C CNN
-	1    5700 2200
-	1    0    0    -1
-$EndComp
-Wire Wire Line
-	6200 2200 6500 2200
+P 5750 2200
+F 0 "DA1" H 5750 2650 60  0000 C CNN
+F 1 "TLV3691" H 5750 2550 60  0000 C CNN
+F 2 "SOT,_TO:SOT353" H 5750 1850 60  0001 C CNN
+F 3 "" H 5750 1850 60  0000 C CNN
+	1    5750 2200
+	1    0    0    -1
+$EndComp
+Wire Wire Line
+	6250 2200 6550 2200
 $Comp
 L Capacitors:C_0603 C5
 U 1 1 633D54D3
-P 6850 2900
-F 0 "C5" H 7000 3100 60  0000 C CNN
-F 1 "0.1u" H 7000 3000 60  0000 C CNN
-F 2 "Capacitors:CAP0603" H 7050 2800 60  0001 C CNN
-F 3 "" H 6850 3150 60  0000 C CNN
-	1    6850 2900
-	1    0    0    -1
-$EndComp
-Wire Wire Line
-	6850 2650 6850 2200
+P 6900 2900
+F 0 "C5" H 7050 3100 60  0000 C CNN
+F 1 "0.1u" H 7050 3000 60  0000 C CNN
+F 2 "Capacitors:CAP0603" H 7100 2800 60  0001 C CNN
+F 3 "" H 6900 3150 60  0000 C CNN
+	1    6900 2900
+	1    0    0    -1
+$EndComp
+Wire Wire Line
+	6900 2650 6900 2200
 $Comp
 L Power:GND #PWR07
 U 1 1 633D54DE
-P 6850 3250
-F 0 "#PWR07" H 6940 3230 30  0001 C CNN
-F 1 "GND" H 6850 3170 30  0001 C CNN
-F 2 "" H 6850 3250 60  0001 C CNN
-F 3 "" H 6850 3250 60  0001 C CNN
-	1    6850 3250
-	1    0    0    -1
-$EndComp
-Wire Wire Line
-	6850 3150 6850 3250
-Wire Wire Line
-	6250 2400 6250 3250
+P 6900 3250
+F 0 "#PWR07" H 6990 3230 30  0001 C CNN
+F 1 "GND" H 6900 3170 30  0001 C CNN
+F 2 "" H 6900 3250 60  0001 C CNN
+F 3 "" H 6900 3250 60  0001 C CNN
+	1    6900 3250
+	1    0    0    -1
+$EndComp
+Wire Wire Line
+	6900 3150 6900 3250
+Wire Wire Line
+	6300 2400 6300 3250
 $Comp
 L Power:GND #PWR05
 U 1 1 633D54EA
-P 6250 3250
-F 0 "#PWR05" H 6340 3230 30  0001 C CNN
-F 1 "GND" H 6250 3170 30  0001 C CNN
-F 2 "" H 6250 3250 60  0001 C CNN
-F 3 "" H 6250 3250 60  0001 C CNN
-	1    6250 3250
+P 6300 3250
+F 0 "#PWR05" H 6390 3230 30  0001 C CNN
+F 1 "GND" H 6300 3170 30  0001 C CNN
+F 2 "" H 6300 3250 60  0001 C CNN
+F 3 "" H 6300 3250 60  0001 C CNN
+	1    6300 3250
 	1    0    0    -1
 $EndComp
@@
 L Capacitors:C_0603 C4
 U 1 1 633D54F4
-P 6500 2900
-F 0 "C4" H 6650 3100 60  0000 C CNN
-F 1 "1n" H 6650 3000 60  0000 C CNN
-F 2 "Capacitors:CAP0603" H 6700 2800 60  0001 C CNN
-F 3 "" H 6500 3150 60  0000 C CNN
-	1    6500 2900
+P 6550 2900
+F 0 "C4" H 6700 3100 60  0000 C CNN
+F 1 "1n" H 6700 3000 60  0000 C CNN
+F 2 "Capacitors:CAP0603" H 6750 2800 60  0001 C CNN
+F 3 "" H 6550 3150 60  0000 C CNN
+	1    6550 2900
 	1    0    0    -1
 $EndComp
@@
 L Power:GND #PWR06
 U 1 1 633D54FE
-P 6500 3250
-F 0 "#PWR06" H 6590 3230 30  0001 C CNN
-F 1 "GND" H 6500 3170 30  0001 C CNN
-F 2 "" H 6500 3250 60  0001 C CNN
-F 3 "" H 6500 3250 60  0001 C CNN
-	1    6500 3250
-	1    0    0    -1
-$EndComp
-Wire Wire Line
-	6500 2650 6500 2200
-Connection ~ 6500 2200
-Wire Wire Line
-	6500 2200 6850 2200
-Wire Wire Line
-	6500 3250 6500 3150
-Wire Wire Line
-	6950 2200 6850 2200
-Connection ~ 6850 2200
+P 6550 3250
+F 0 "#PWR06" H 6640 3230 30  0001 C CNN
+F 1 "GND" H 6550 3170 30  0001 C CNN
+F 2 "" H 6550 3250 60  0001 C CNN
+F 3 "" H 6550 3250 60  0001 C CNN
+	1    6550 3250
+	1    0    0    -1
+$EndComp
+Wire Wire Line
+	6550 2650 6550 2200
+Connection ~ 6550 2200
+Wire Wire Line
+	6550 2200 6900 2200
+Wire Wire Line
+	6550 3250 6550 3150
+Wire Wire Line
+	7000 2200 6900 2200
+Connection ~ 6900 2200
 $Comp
 L Power:GND #PWR03
@@
 Wire Wire Line
 	3850 1050 3050 1050
-Text Label 6950 2200 0    60   ~ 0
+Text Label 7000 2200 0    60   ~ 0
 +LightSns_PWR
-Text Label 7000 2000 0    60   ~ 0
+Text Label 7050 2000 0    60   ~ 0
 LightSns_OUT
 $Comp
 L Capacitors:C_0603 C3
 U 1 1 634452D6
-P 5150 2850
-F 0 "C3" H 5300 3050 60  0000 C CNN
-F 1 "0.1uF" H 5300 2950 60  0000 C CNN
-F 2 "Capacitors:CAP0603" H 5350 2750 60  0001 C CNN
-F 3 "" H 5150 3100 60  0000 C CNN
-	1    5150 2850
-	1    0    0    -1
-$EndComp
-Wire Wire Line
-	6200 2000 6250 2000
+P 5200 2850
+F 0 "C3" H 5350 3050 60  0000 C CNN
+F 1 "0.1u" H 5350 2950 60  0000 C CNN
+F 2 "Capacitors:CAP0603" H 5400 2750 60  0001 C CNN
+F 3 "" H 5200 3100 60  0000 C CNN
+	1    5200 2850
+	1    0    0    -1
+$EndComp
+Wire Wire Line
+	6250 2000 6300 2000
 Connection ~ 6700 5000
 $Comp
@@
 $EndComp
 Wire Wire Line
-	5150 1050 5150 1550
-Connection ~ 5150 1550
-Wire Wire Line
-	5150 1550 5150 2000
+	5200 1050 5200 1550
+Connection ~ 5200 1550
+Wire Wire Line
+	5200 1550 5200 2000
 $Comp
 L Power:GND #PWR04
 U 1 1 63453F5E
-P 5150 3250
-F 0 "#PWR04" H 5240 3230 30  0001 C CNN
-F 1 "GND" H 5150 3170 30  0001 C CNN
-F 2 "" H 5150 3250 60  0001 C CNN
-F 3 "" H 5150 3250 60  0001 C CNN
-	1    5150 3250
-	1    0    0    -1
-$EndComp
-Wire Wire Line
-	5150 3250 5150 3100
-Wire Wire Line
-	6250 2000 6250 1550
-Wire Wire Line
-	5950 1050 6250 1050
-Connection ~ 6250 2000
-Wire Wire Line
-	6250 2000 7000 2000
-Connection ~ 6250 1550
-Wire Wire Line
-	6250 1550 6250 1050
-Wire Wire Line
-	6250 2400 6200 2400
-Connection ~ 5150 2000
-Wire Wire Line
-	5150 2000 4700 2000
-Wire Wire Line
-	5150 2000 5150 2600
+P 5200 3250
+F 0 "#PWR04" H 5290 3230 30  0001 C CNN
+F 1 "GND" H 5200 3170 30  0001 C CNN
+F 2 "" H 5200 3250 60  0001 C CNN
+F 3 "" H 5200 3250 60  0001 C CNN
+	1    5200 3250
+	1    0    0    -1
+$EndComp
+Wire Wire Line
+	5200 3250 5200 3100
+Wire Wire Line
+	6300 2000 6300 1550
+Wire Wire Line
+	6000 1050 6300 1050
+Connection ~ 6300 2000
+Wire Wire Line
+	6300 2000 7050 2000
+Connection ~ 6300 1550
+Wire Wire Line
+	6300 1550 6300 1050
+Wire Wire Line
+	6300 2400 6250 2400
+Connection ~ 5200 2000
+Wire Wire Line
+	5200 2000 4700 2000
+Wire Wire Line
+	5200 2000 5200 2600
 $Comp
 L Resistors:R_TRIM R1
@@
 P 4250 1050
 F 0 "R1" H 4100 1350 60  0000 C CNN
-F 1 "100k" H 4100 1250 60  0000 C CNN
+F 1 "10M" H 4100 1250 60  0000 C CNN
 F 2 "Resistors:RES_TRIM_Bourns3314J-1" H 3850 1050 60  0001 C CNN
 F 3 "" H 3850 1050 60  0000 C CNN
